File: ice-samd.sch (KiCad schematic (older format))
At the start: 26 parts, among them J1 Conn_Battery, J2 USB_B_Micro, J3 Conn_Left, J4 Conn_Right, U1 SPX3819M5-L-3-3, U2 ATSAMD21G18A-AUT, U3 MCP73831-2-OT, Y1 32.768

Commit message: Updated samd21
Parts:
- added IC1: ADXL345, ADX:ADXL3x5, symbol ADX:ADXL345
- added R7, R8: 10k, Resistor_SMD:R_0603_1608Metric, symbol Device:R_Small
- added U4: ATECC608A-MAHDA, Package_DFN_QFN:DFN-8-1EP_3x2mm_P0.5mm_EP1.3x1.5mm, symbol Security:ATECC608A-MAHDA
Connections:
- net +3V3: now also IC1.1 (VDD_IO), IC1.6 (Vs), IC1.7 (CS), R7.2, R8.2, U4.8 (VCC)
- net GND: now also IC1.13 (SDI), IC1.2 (GND), IC1.4 (GND), IC1.5 (GND), U4.4 (GND)
- net SCL: now also IC1.14 (SCLK), R8.1, U4.6 (SCL)
- net SDA: now also IC1.12 (SDO), R7.1, U4.5 (SDA)
- no-connect marks 3 -> 4
Other:
- moved on the sheet: D3, R4, R5, R6
